Commit message: カメラモデルを変更しやすいようにファイル構造を変更

File: urdf/hac_camera.xacro (robot description, xacro)
@@ -38,45 +38,4 @@
       <parent link="camera_pole"/>
     </joint>
-    <gazebo reference="camera_link">
-      <material>Gazebo/Red</material>
-      <sensor type="camera" name="camera1">
-        <update_rate>30.0</update_rate>
-        <camera name="head">
-          <!-- 視野角 -->
-          <!-- 55deg = 0.9599 rad -->
-          <horizontal_fov>0.9599</horizontal_fov>
-          <!-- 解像度とフォーマット -->
-          <image>
-            <width>1280</width>
-            <height>720</height>
-            <format>R8G8B8</format>
-            <!-- <format>B8G8R8</format> -->
-          </image>
-          <!-- どれだけの範囲（距離）を認識できるか -->
-          <clip>
-            <near>0.02</near>
-            <far>300</far>
-          </clip>
-          <!-- ノイズを大きくすれば、ノイズに強いプログラムを作れる -->
-          <noise>
-            <type>gaussian</type>
-            <!-- Noise is sampled independently per pixel on each frame.
-                That pixel's noise value is added to each of its color
-                channels, which at that point lie in the range [0,1]. -->
-            <mean>0.0</mean>
-            <stddev>0.007</stddev>
-          </noise>
-        </camera>
-        <plugin name="camera_controller" filename="libgazebo_ros_camera.so">
-          <camera_name>c270n</camera_name>
-          <frame_name>camera_link</frame_name>
-          <!-- <distortionK1>0.0</distortionK1>
-          <distortionK2>0.0</distortionK2>
-          <distortionK3>0.0</distortionK3>
-          <distortionT1>0.0</distortionT1>
-          <distortionT2>0.0</distortionT2> -->
-        </plugin>
-      </sensor>
-    </gazebo>
   </xacro:macro>
 </robot>

File: urdf/raspimouse.urdf.xacro (robot description, xacro)
@@ -22,4 +22,5 @@
   <xacro:include filename="$(find raspimouse_description)/urdf/raspimouse.gazebo_ros2_control.xacro" />
   <xacro:include filename="$(find raspimouse_description)/urdf/hac_camera.xacro" />
+  <xacro:include filename="$(find raspimouse_description)/urdf/camera_c270n.xacro" />
   <!-- =============== Link & Joint =============== -->
   <!-- Base -->
@@ -67,4 +68,6 @@
       <origin xyz="0.0 0.0 0.2" rpy="0 0 0"/>
     </xacro:hac_camera>
+    <!-- ここで好きなカメラをコメント解除で選択する -->
+    <xacro:camera_c270n/>
   </xacro:if>
   <!-- <xacro:if value="$(arg gazebo_plugin)">

Commit message: カメラを30度下に向けた

File: urdf/hac_camera.xacro (robot description, xacro)
@@ -34,5 +34,5 @@
     </link>
     <joint type="fixed" name="camera_joint">
-      <origin xyz="0.05 0.0 0.05" rpy="0 0 0"/>
+      <origin xyz="0.05 0.0 0.05" rpy="0 0.5236 0"/>
       <child link="camera_link"/>
       <parent link="camera_pole"/>
