Commit message: Add c270n camera

File: urdf/raspimouse.urdf.xacro (robot description, xacro)
@@ -21,4 +21,5 @@
   <xacro:include filename="$(find raspimouse_description)/urdf/sensors/lrf.urdf.xacro" />
   <xacro:include filename="$(find raspimouse_description)/urdf/raspimouse.gazebo_ros2_control.xacro" />
+  <xacro:include filename="$(find raspimouse_description)/urdf/hac_camera.xacro" />
   <!-- =============== Link & Joint =============== -->
   <!-- Base -->
@@ -62,4 +63,8 @@
       config_file_package="hac_demo_bots"
       config_file_path="config/gazebo_controllers.yaml" />
+    <xacro:hac_camera
+      parent="base_link">
+      <origin xyz="0.0 0.0 0.2" rpy="0 0 0"/>
+    </xacro:hac_camera>
   </xacro:if>
   <!-- <xacro:if value="$(arg gazebo_plugin)">

Commit message: カメラの高さが0.35 mになるように調整した

File: urdf/raspimouse.urdf.xacro (robot description, xacro)
@@ -67,5 +67,5 @@
     <xacro:hac_camera
       parent="base_link">
-      <origin xyz="0.0 0.0 0.2" rpy="0 0 0"/>
+      <origin xyz="0.0 0.0 0.3" rpy="0 0 0"/>
     </xacro:hac_camera>
     <!-- ここで好きなカメラをコメント解除で選択する -->
